Commit message: feat(sdf): add sdf support and meshes for sdf robot model

File: src/mlr_nav2_puzzlebot/urdf/puzzlebot.urdf (robot description, URDF)
Before this commit: robot puzzlebot, 5 links, 4 joints
Links:
- link base_footprint: mass None -> 0.01
- link base_link: geometry visual mesh filename=package://mlr_nav2_puzzlebot/meshes/Puzzlebot_Jetson_Lidar_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
- link caster: geometry visual mesh filename=package://mlr_nav2_puzzlebot/meshes/Puzzlebot_Caster_Wheel.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
- link wheel_l: mass None -> 0.1; geometry visual mesh filename=package://mlr_nav2_puzzlebot/meshes/Puzzlebot_Wheel.stl
- link wheel_r: mass None -> 0.1; geometry visual mesh filename=package://mlr_nav2_puzzlebot/meshes/Puzzlebot_Wheel.stl

Commit message: Change URDF

File: src/mlr_nav2_puzzlebot/urdf/puzzlebot.urdf (robot description, URDF)
Before this commit: robot puzzlebot, 5 links, 4 joints
Links:
- link base_link: mass None -> 2.0; geometry collision mesh filename=package://mlr_nav2_puzzlebot/meshes/Puzzlebot_Jetson_Lidar_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; visual mesh filename=package://mlr_nav2_puzzlebot/meshes/Puzzlebot_Jetson_Lidar_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
- link caster: mass None -> 0.001; geometry collision mesh filename=package://mlr_nav2_puzzlebot/meshes/Puzzlebot_Caster_Wheel.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; visual mesh filename=package://mlr_nav2_puzzlebot/meshes/Puzzlebot_Caster_Wheel.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
- link wheel_l: mass 0.1 -> 0.2; geometry collision mesh filename=package://mlr_nav2_puzzlebot/meshes/Puzzlebot_Wheel.stl; visual mesh filename=package://mlr_nav2_puzzlebot/meshes/Puzzlebot_Wheel.stl
- link wheel_r: mass 0.1 -> 0.2; geometry collision mesh filename=package://mlr_nav2_puzzlebot/meshes/Puzzlebot_Wheel.stl; visual mesh filename=package://mlr_nav2_puzzlebot/meshes/Puzzlebot_Wheel.stl
